File: STM32.kicad_sch (KiCad schematic)
At the start: 28 parts, among them J1 USB_C_Receptacle_USB2.0_16P, SW1 SW_SPST, SW2 SW_SPST, U2 ADUM4160, U7 USBLC6-2SC6, U8 DS8572-33S5, U9 STM32F072CBTx

Commit message: draf 1 for sims
Connections:
- net A4 renamed PA4
- net A5 renamed PA5
- net A6: no longer names the net of U9.16 (PA6)
- net A7 renamed PA7
- net B0 renamed PB0
- net B12 renamed PB12
- net B13 renamed PB13
- net B14 renamed PB14
- net B15 renamed PB15

Commit message: current routing stage
Parts:
- C24, C25, C26, C27: footprint (none) -> Capacitor_SMD:C_0805_2012Metric
- J1: footprint My Parts Library:USB-C-16-Pin-MidMount -> Connector_USB:USB_C_Receptacle_Molex_105450-0101
Changed lines of the file:
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@@
 			)
 		)
-		(property "Footprint" ""
+		(property "Footprint" "Capacitor_SMD:C_0805_2012Metric"
 			(at 110.7948 40.64 0)
 			(effects
@@
 			)
 		)
-		(property "Footprint" ""
+		(property "Footprint" "Capacitor_SMD:C_0805_2012Metric"
 			(at 113.03 54.3052 0)
 			(effects
@@
 			)
 		)
-		(property "Footprint" "My Parts Library:USB-C-16-Pin-MidMount"
+		(property "Footprint" "Connector_USB:USB_C_Receptacle_Molex_105450-0101"
 			(at 43.18 58.42 0)
 			(effects
@@
 			)
 		)
-		(property "Footprint" ""
+		(property "Footprint" "Capacitor_SMD:C_0805_2012Metric"
 			(at 89.2048 44.45 0)
 			(effects
@@
 			)
 		)
-		(property "Footprint" ""
+		(property "Footprint" "Capacitor_SMD:C_0805_2012Metric"
 			(at 120.65 59.3852 0)
 			(effects

Commit message: sim the new lpf
Parts:
- removed TP1, TP2: TestPoint, TestPoint:TestPoint_Pad_1.5x1.5mm, symbol Connector:TestPoint
- added R27, R28, R29, R30: 24, Resistor_SMD:R_0201_0603Metric, symbol Device:R
- C13, C14, C15, C16, C17, C18, C19, C20, C21, C22, C23, C24, C25, C26, C27: footprint Capacitor_SMD:C_0805_2012Metric -> Capacitor_SMD:C_0201_0603Metric
- J1: footprint Connector_USB:USB_C_Receptacle_Molex_105450-0101 -> Connector_USB:USB_C_Receptacle_GCT_USB4105-xx-A_16P_TopMnt_Horizontal
- R15, R16: footprint Resistor_SMD:R_0805_2012Metric -> Resistor_SMD:R_0201_0603Metric
Connections:
- net +5V: now also C27.2, U2.16 (VBUS2); no longer C24.1, F1.1, U2.3 (VDD1), U2.4 (PDEN), U2.5 (SPU)
- net D+: now also R28.2; no longer J1.A6 (D+), J1.B6 (D+)
- net D+iso: now also R30.2; no longer U2.10 (DD+)
- net D-: now also R27.2; no longer J1.A7 (D-), J1.B7 (D-)
- net D-iso: now also R29.2; no longer U2.11 (DD-)
- net GND: no longer U2.13 (SPD)
- net VBUS: no longer C25.1, U2.1 (VBUS1)
- net at C26.2, U2.14 (VDD2): now also U2.13 (SPD)
- new net: C25.1, F1.1, U2.1 (VBUS1)
- new net: J1.A7 (D-), J1.B7 (D-), R27.1
- new net: R30.1, U2.10 (DD+)
- new net: J1.A6 (D+), J1.B6 (D+), R28.1
- new net: R29.1, U2.11 (DD-)
- new net: C24.1, U2.3 (VDD1), U2.4 (PDEN), U2.5 (SPU)
