File: Wavegen_esb.kicad_sch (KiCad schematic)
At the start: 14 parts, among them IC1 PA107DP, U5 LMH6881SQ/NOPB

Commit message: test
Parts:
- R13: value 2.6k -> 1k
Changed lines of the file:
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@@
 			)
 		)
-		(property "Value" "2.6k"
+		(property "Value" "1k"
 			(at 166.37 33.02 0)
 			(effects

Commit message: pa107 wiring 1
Parts:
- removed IC1: PA107DP, PA107DP, symbol PA107DP:PA107DP
- added C45: 10uf, symbol Device:C
- added J3: Screw_Terminal_01x02, symbol Connector:Screw_Terminal_01x02
- R13: value 1k -> 2.6k
Connections:
- net +out renamed PA107/PA_IN
- net -out renamed PA108/PA_IN
- new net: C45.1, J3.1 (Pin_1), J3.2 (Pin_2)
- new net PA107/PA107OUT: C45.2
- no-connect marks 6 -> 3
Other:
- added sheet 5v (5v.kicad_sch)
- added sheet PA107 (PA107.kicad_sch)
- added sheet PA108 (PA107.kicad_sch)
- moved on the sheet: C12, R11, R12, R13

Commit message: draf 1 for sims
Parts:
- removed C10, C11, C12: 0.1pf, symbol Device:C
- removed C28: 4.7uf, symbol Device:C
- removed R10: 1k, symbol Device:R
- removed R11, R14, R18: 50, symbol Device:R
- removed R12, R13: 2.6k, symbol Device:R
- removed R19: 400, symbol Device:R
- removed R9: 3k, symbol Device:R
- removed U5: LMH6881SQ/NOPB, RTW0024A, symbol 1_variable gain:LMH6881SQ_NOPB
- added C50, C52: 100nf, symbol Device:C
- added C51, C53: 10uf, symbol Device:C
- added U11, U12, U13: ~, 1_Sockets:Untitled, symbol 1_variable gain:1_4mm_SOCKET
Connections:
- net GND: now also C50.2, C51.2, C52.2, C53.2, U13.1, U13.2
- net at C45.1, J3.1 (Pin_1): no longer J3.2 (Pin_2)
- new net: C52.1, C53.1, U11.1, U11.2
- new net -5V: C50.1, C51.1, U12.1, U12.2
- new net PA108/PA107OUT: J3.2 (Pin_2)
- no-connect marks 3 -> 0
Other:
- added sheet VGA (VGA.kicad_sch)
- sheet PA107 ports: added +Vs, +vaux, -Vs, -vaux; removed none
- sheet PA108 ports: added +Vs, +vaux, -Vs, -vaux; removed none
- sheet STM32 ports: added PA4, PA5, PA7, PB0, PB12, PB13, PB14, PB15; removed none
- sheet dds ports: added FSYNC, MCLK, RESET, SCLK, SDATA, SIGNAL; removed none
- moved on the sheet: C45, J3

Commit message: current routing stage
Parts:
- removed C50, C52: 100nf, symbol Device:C
- removed C51, C53: 10uf, symbol Device:C
- removed J3: Screw_Terminal_01x02, symbol Connector:Screw_Terminal_01x02
- removed U11, U12, U13: ~, 1_Sockets:Untitled, symbol 1_variable gain:1_4mm_SOCKET
- added J3: 2601-1102, lever_terminal:CONN2_2601-1102_WAG, symbol lever_terminal:2601-1102
- C45: footprint (none) -> Capacitor_SMD:C_0805_2012Metric
Connections:
- net PA108/PA107OUT: now also J3.3 (2_1)
- net at C45.1: now also J3.2 (1_2)
Other:
- removed sheet 5v
- added sheet power (power.kicad_sch)

Commit message: sim the new lpf
Parts:
- C45: footprint Capacitor_SMD:C_0805_2012Metric -> 1_cap:CAPRR1500W80L2600T1150H2600
Changed lines of the file:
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@@
 			)
 		)
-		(property "Footprint" "Capacitor_SMD:C_0805_2012Metric"
+		(property "Footprint" "1_cap:CAPRR1500W80L2600T1150H2600"
 			(at 264.16 100.0252 0)
 			(effects
