File: VGA.kicad_sch (KiCad schematic)
At the start: 13 parts, among them U5 LMH6881SQ/NOPB

Commit message: current routing stage
Parts:
- added C58, C59: 4.7uf, Capacitor_SMD:C_0805_2012Metric, symbol Device:C
- C10, C11, C12, C28, R11, R12, R13, R19, R9: footprint (none) -> Capacitor_SMD:C_0805_2012Metric
- R10: footprint (none) -> Resistor_SMD:R_0805_2012Metric
- R14, R18: value 50 -> 1k; footprint (none) -> Resistor_SMD:R_0805_2012Metric
- U5: footprint RTW0024A -> 1_variable gain:RTW0024A
Connections:
- net OUTM: now also C59.1; no longer R18.2
- net OUTP: now also C58.1; no longer R14.2
- new net: C58.2, R14.2
- new net: C59.2, R18.2
Changed lines of the file:
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@@
 	(hierarchical_label "OUTM"
 		(shape input)
-		(at 151.13 101.6 0)
+		(at 158.75 101.6 0)
 		(effects
 			(font
@@
 	(hierarchical_label "OUTP"
 		(shape input)
-		(at 151.13 91.44 0)
+		(at 158.75 91.44 0)
 		(effects
 			(font
@@
 			)
 		)
-		(property "Footprint" ""
+		(property "Footprint" "Capacitor_SMD:C_0805_2012Metric"
 			(at 138.7348 77.47 0)
 			(effects
@@
 	)
 	(symbol
+		(lib_id "Device:C")
+		(at 154.94 91.44 270)
+		(unit 1)
+		(exclude_from_sim no)
+		(in_bom yes)
+		(on_board yes)
+		(dnp no)
+		(fields_autoplaced yes)
+		(property "Reference" "C58"
+			(at 154.94 83.82 90)
+			(effects
+				(font
+					(size 1.27 1.27)
+				)
+			)
+		)
+		(property "Value" "4.7uf"
+			(at 154.94 86.36 90)
+			(effects
+				(font
+					(size 1.27 1.27)
+				)
+			)
+		)
+		(property "Footprint" "Capacitor_SMD:C_0805_2012Metric"
+			(at 151.13 92.4052 0)
+			(effects
+				(font
+					(size 1.27 1.27)
+				)
+				(hide yes)
+			)
+		)
+		(property "Datasheet" "~"
+			(at 154.94 91.44 0)
+			(effects
+				(font
+					(size 1.27 1.27)
+				)
+				(hide yes)
+			)
+		)
+		(property "Description" "Unpolarized capacitor"
+			(at 154.94 91.44 0)
+			(effects
+				(font
+					(size 1.27 1.27)
+				)
+				(hide yes)
+			)
+		)
+		(pin "2"
+		)
+		(pin "1"
+		)
+		(instances
+			(project "Wavegen_esb"
+				(path "/83dee5c5-8c71-4ecf-8c4b-74a6ca3f5e87/ae7dc586-15c3-4753-ac70-eec13d02e883"
+					(reference "C58")
+					(unit 1)
+				)
+			)
+		)
+	)
+	(symbol
 		(lib_id "Device:R")
 		(at 147.32 101.6 90)
@@
 			)
 		)
-		(property "Value" "50"
+		(property "Value" "1k"
 			(at 147.32 97.79 90)
 			(effects
@@
 			)
 		)
-		(property "Footprint" ""
+		(property "Footprint" "Resistor_SMD:R_0805_2012Metric"
 			(at 147.32 103.378 90)
 			(effects
@@
 			)
 		)
+		(property "Field5" ""
+			(at 147.32 101.6 90)
+			(effects
+				(font
+					(size 1.27 1.27)
+				)
+				(hide yes)
+			)
+		)
 		(pin "1"
 		)
@@
 			)
 		)
-		(property "Footprint" ""
+		(property "Footprint" "Capacitor_SMD:C_0805_2012Metric"
 			(at 122.682 53.34 90)
 			(effects
@@
 			)
 		)
-		(property "Footprint" ""
+		(property "Footprint" "Resistor_SMD:R_0805_2012Metric"
 			(at 84.582 62.23 90)
 			(effects
@@
 			)
 		)
-		(property "Footprint" ""
+		(property "Footprint" "Capacitor_SMD:C_0805_2012Metric"
 			(at 84.582 54.61 90)
 			(effects
@@
 				(path "/83dee5c5-8c71-4ecf-8c4b-74a6ca3f5e87/ae7dc586-15c3-4753-ac70-eec13d02e883"
 					(reference "R9")
+					(unit 1)
+				)
+			)
+		)
+	)
+	(symbol
+		(lib_id "Device:C")
+		(at 154.94 101.6 270)
+		(unit 1)
+		(exclude_from_sim no)
+		(in_bom yes)
+		(on_board yes)
+		(dnp no)
+		(fields_autoplaced yes)
+		(property "Reference" "C59"
+			(at 154.94 93.98 90)
+			(effects
+				(font
+					(size 1.27 1.27)
+				)
+			)
+		)
+		(property "Value" "4.7uf"
+			(at 154.94 96.52 90)
+			(effects
+				(font
+					(size 1.27 1.27)
+				)
+			)
+		)
+		(property "Footprint" "Capacitor_SMD:C_0805_2012Metric"
+			(at 151.13 102.5652 0)
+			(effects
+				(font
+					(size 1.27 1.27)
+				)
+				(hide yes)
+			)
+		)
+		(property "Datasheet" "~"
+			(at 154.94 101.6 0)
+			(effects
+				(font
+					(size 1.27 1.27)
+				)
+				(hide yes)
+			)
+		)
+		(property "Description" "Unpolarized capacitor"
+			(at 154.94 101.6 0)
+			(effects
+				(font
+					(size 1.27 1.27)
+				)
+				(hide yes)
+			)
+		)
+		(pin "2"
+		)
+		(pin "1"
+		)
+		(instances
+			(project "Wavegen_esb"
+				(path "/83dee5c5-8c71-4ecf-8c4b-74a6ca3f5e87/ae7dc586-15c3-4753-ac70-eec13d02e883"
+					(reference "C59")
 					(unit 1)
 				)
@@
 			)
 		)
-		(property "Footprint" ""
+		(property "Footprint" "Capacitor_SMD:C_0805_2012Metric"
 			(at 111.76 90.4748 0)
 			(effects
@@
 			)
 		)
-		(property "Footprint" ""
+		(property "Footprint" "Capacitor_SMD:C_0805_2012Metric"
 			(at 136.1948 57.15 0)
 			(effects
@@
 			)
 		)
-		(property "Value" "50"
+		(property "Value" "1k"
 			(at 147.32 87.63 90)
 			(effects
@@
 			)
 		)
-		(property "Footprint" ""
+		(property "Footprint" "Resistor_SMD:R_0805_2012Metric"
 			(at 147.32 93.218 90)
 			(effects
@@
 			)
 		)
-		(property "Footprint" "RTW0024A"
+		(property "Footprint" "1_variable gain:RTW0024A"
 			(at 124.46 137.16 0)
 			(effects
@@
 			)
 		)
-		(property "Footprint" "RTW0024A"
+		(property "Footprint" "1_variable gain:RTW0024A"
 			(at 124.46 96.52 0)
 			(effects
@@
 			)
 		)
-		(property "Footprint" ""
+		(property "Footprint" "Capacitor_SMD:C_0805_2012Metric"
 			(at 122.682 60.96 90)
 			(effects
@@
 			)
 		)
-		(property "Footprint" ""
+		(property "Footprint" "Capacitor_SMD:C_0805_2012Metric"
 			(at 96.8248 58.42 0)
 			(effects
@@
 			)
 		)
-		(property "Footprint" ""
+		(property "Footprint" "Capacitor_SMD:C_0805_2012Metric"
 			(at 135.382 53.34 90)
 			(effects
@@
 			)
 		)
-		(property "Footprint" ""
+		(property "Footprint" "Capacitor_SMD:C_0805_2012Metric"
 			(at 99.822 120.65 90)
 			(effects

Commit message: sim the new lpf
Parts:
- C10: value 0.1pf -> 0.1uf; footprint Capacitor_SMD:C_0805_2012Metric -> Capacitor_SMD:C_0201_0603Metric
- C11, C12: value 0.1pf -> 10uf; footprint Capacitor_SMD:C_0805_2012Metric -> Capacitor_SMD:C_0201_0603Metric
- C28: value 4.7uf -> 1uf; footprint Capacitor_SMD:C_0805_2012Metric -> Capacitor_SMD:C_0201_0603Metric
- R10: footprint Resistor_SMD:R_0805_2012Metric -> Resistor_SMD:R_0201_0603Metric
- R11, R12, R13, R19, R9: footprint Capacitor_SMD:C_0805_2012Metric -> Resistor_SMD:R_0201_0603Metric
- R14, R18: value 1k -> 665
Connections:
- net +5V: now also U5.5 (SPI)
- net GND: now also C12.2; no longer C12.1
- net at R11.2, R12.2, R13.1: now also C12.1; no longer C12.2
Other:
- moved on the sheet: C12
Changed lines of the file:
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@@
-	)
-	(junction
-		(at 137.16 57.15)
-		(diameter 0)
-		(color 0 0 0 0)
 	)
 	(junction
@@
 	(junction
 		(at 129.54 106.68)
+		(diameter 0)
+		(color 0 0 0 0)
+	)
+	(junction
+		(at 137.16 57.15)
 		(diameter 0)
 		(color 0 0 0 0)
@@
 			)
 		)
-		(property "Value" "0.1pf"
+		(property "Value" "0.1uf"
 			(at 143.51 82.5499 0)
 			(effects
@@
 			)
 		)
-		(property "Footprint" "Capacitor_SMD:C_0805_2012Metric"
+		(property "Footprint" "Capacitor_SMD:C_0201_0603Metric"
 			(at 138.7348 77.47 0)
 			(effects
@@
 	)
 	(symbol
+		(lib_id "power:+5V")
+		(at 106.68 129.54 0)
+		(unit 1)
+		(exclude_from_sim no)
+		(in_bom yes)
+		(on_board yes)
+		(dnp no)
+		(fields_autoplaced yes)
+		(property "Reference" "#PWR0101"
+			(at 106.68 133.35 0)
+			(effects
+				(font
+					(size 1.27 1.27)
+				)
+				(hide yes)
+			)
+		)
+		(property "Value" "+5V"
+			(at 106.68 124.46 0)
+			(effects
+				(font
+					(size 1.27 1.27)
+				)
+			)
+		)
+		(property "Footprint" ""
+			(at 106.68 129.54 0)
+			(effects
+				(font
+					(size 1.27 1.27)
+				)
+				(hide yes)
+			)
+		)
+		(property "Datasheet" ""
+			(at 106.68 129.54 0)
+			(effects
+				(font
+					(size 1.27 1.27)
+				)
+				(hide yes)
+			)
+		)
+		(property "Description" "Power symbol creates a global label with name \"+5V\""
+			(at 106.68 129.54 0)
+			(effects
+				(font
+					(size 1.27 1.27)
+				)
+				(hide yes)
+			)
+		)
+		(pin "1"
+		)
+		(instances
+			(project "Wavegen_esb"
+				(path "/83dee5c5-8c71-4ecf-8c4b-74a6ca3f5e87/ae7dc586-15c3-4753-ac70-eec13d02e883"
+					(reference "#PWR0101")
+					(unit 1)
+				)
+			)
+		)
+	)
+	(symbol
 		(lib_id "power:GND")
 		(at 101.6 124.46 0)
@@
 			)
 		)
-		(property "Value" "1k"
+		(property "Value" "665"
 			(at 147.32 97.79 90)
 			(effects
@@
 			)
 		)
-		(property "Footprint" "Capacitor_SMD:C_0805_2012Metric"
+		(property "Footprint" "Resistor_SMD:R_0201_0603Metric"
 			(at 122.682 53.34 90)
 			(effects
@@
 			)
 		)
-		(property "Footprint" "Resistor_SMD:R_0805_2012Metric"
+		(property "Footprint" "Resistor_SMD:R_0201_0603Metric"
 			(at 84.582 62.23 90)
 			(effects
@@
 			)
 		)
-		(property "Footprint" "Capacitor_SMD:C_0805_2012Metric"
+		(property "Footprint" "Resistor_SMD:R_0201_0603Metric"
 			(at 84.582 54.61 90)
 			(effects
@@
 			)
 		)
-		(property "Value" "4.7uf"
+		(property "Value" "1uf"
 			(at 107.95 86.36 90)
 			(effects
@@
 			)
 		)
-		(property "Footprint" "Capacitor_SMD:C_0805_2012Metric"
+		(property "Footprint" "Capacitor_SMD:C_0201_0603Metric"
 			(at 111.76 90.4748 0)
 			(effects
@@
 	(symbol
 		(lib_id "Device:C")
-		(at 137.16 60.96 180)
+		(at 137.16 60.96 0)
 		(unit 1)
 		(exclude_from_sim no)
@@
 					(size 1.27 1.27)
 				)
-				(justify right)
-			)
-		)
-		(property "Value" "0.1pf"
+				(justify left)
+			)
+		)
+		(property "Value" "10uf"
 			(at 140.97 62.2299 0)
 			(effects
@@
 					(size 1.27 1.27)
 				)
-				(justify right)
-			)
-		)
-		(property "Footprint" "Capacitor_SMD:C_0805_2012Metric"
-			(at 136.1948 57.15 0)
+				(justify left)
+			)
+		)
+		(property "Footprint" "Capacitor_SMD:C_0201_0603Metric"
+			(at 138.1252 64.77 0)
 			(effects
 				(font
@@
 			)
 		)
-		(property "Value" "1k"
+		(property "Value" "665"
 			(at 147.32 87.63 90)
 			(effects
@@
 			)
 		)
-		(property "Footprint" "Capacitor_SMD:C_0805_2012Metric"
+		(property "Footprint" "Resistor_SMD:R_0201_0603Metric"
 			(at 122.682 60.96 90)
 			(effects
@@
 			)
 		)
-		(property "Value" "0.1pf"
+		(property "Value" "10uf"
 			(at 101.6 63.4999 0)
 			(effects
@@
 			)
 		)
-		(property "Footprint" "Capacitor_SMD:C_0805_2012Metric"
+		(property "Footprint" "Capacitor_SMD:C_0201_0603Metric"
 			(at 96.8248 58.42 0)
 			(effects
@@
 			)
 		)
-		(property "Footprint" "Capacitor_SMD:C_0805_2012Metric"
+		(property "Footprint" "Resistor_SMD:R_0201_0603Metric"
 			(at 135.382 53.34 90)
 			(effects
@@
 			)
 		)
-		(property "Footprint" "Capacitor_SMD:C_0805_2012Metric"
+		(property "Footprint" "Resistor_SMD:R_0201_0603Metric"
 			(at 99.822 120.65 90)
 			(effects

Commit message: routing draft 2
Parts:
- added C60, C7: 0.1uF, Capacitor_SMD:C_0201_0603Metric, symbol Device:C
- added C61, C9: 10uf, Capacitor_THT:C_Radial_D5.0mm_H5.0mm_P2.00mm, symbol Device:C
- added C62, C63: 100pF, Capacitor_SMD:C_0805_2012Metric, symbol Device:C
- added R31, R32: 1k, Resistor_SMD:R_0805_2012Metric, symbol Device:R
- added R33, R6: 5k, Resistor_SMD:R_0805_2012Metric, symbol Device:R
- added R4, R5: 100k, Resistor_SMD:R_0805_2012Metric, symbol Device:R
- added U4: OPA2192IDR, DGK0008A_N_TEX, symbol 1_preamp:OPA2192IDR
Connections:
- net GND: now also C60.2, C61.2, C62.2, C63.2, C7.2, C9.2, R31.1, R32.1, R4.2, R5.2
- net OUTM: now also R33.2, U4.7 (OUT); no longer C59.1
- net OUTP: now also R6.2, U4.1 (OUT); no longer C58.1
- net at R14.2: now also C63.1, U4.5 (IN+); no longer C58.2
- net at R18.1: now also C59.1, R4.1; no longer U5.21 (OUTM)
- net at R18.2: now also C62.1, U4.3 (IN+); no longer C59.2
- net at R14.1: now also C58.1, R5.1; no longer U5.22 (OUTP)
- new net: C58.2, U5.22 (OUTP)
- new net: C59.2, U5.21 (OUTM)
- new net +V: C60.1, C61.1, U4.8 (V+)
- new net -INa: R31.2, R6.1, U4.2 (IN-)
- new net -INb: R32.2, R33.1, U4.6 (IN-)
- new net -V: C7.1, C9.1, U4.4 (V-)
Other:
- moved on the sheet: C58, C59, R14, R18
