File: PA107.kicad_sch (KiCad schematic)
At the start: 10 parts, among them IC1 PA107DP

Commit message: draf 1 for sims
Parts:
- added R22, R23: 47k, symbol Device:R
Connections:
- net +Vsp is gone; now on net +Vs: C34.2, C35.2
- net GND: now also R22.1, R23.1
- net +55V renamed +Vs
- net +Vs: now also R23.2
- net -55V renamed -Vs
- net -Vs: now also R22.2

Commit message: current routing stage
Parts:
- C29, C30, C31, C32, C33, C34: footprint (none) -> Capacitor_SMD:C_0805_2012Metric
- C35, C36: footprint (none) -> Capacitor_THT:CP_Radial_D6.3mm_P2.50mm
- IC1: footprint PA107DP -> pa107:PA107DP
- R20, R23: footprint (none) -> Resistor_SMD:R_0805_2012Metric
- R47: renamed from R22; footprint (none) -> Resistor_SMD:R_0805_2012Metric
Changed lines of the file:
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@@
 			)
 		)
-		(property "Footprint" ""
+		(property "Footprint" "Resistor_SMD:R_0805_2012Metric"
 			(at 163.068 52.07 90)
 			(effects
@@
 			)
 		)
-		(property "Footprint" ""
+		(property "Footprint" "Capacitor_SMD:C_0805_2012Metric"
 			(at 104.4448 29.21 0)
 			(effects
@@
 		(dnp no)
 		(fields_autoplaced yes)
-		(property "Reference" "R22"
+		(property "Reference" "R47"
 			(at 165.1 31.7499 0)
 			(effects
@@
 			)
 		)
-		(property "Footprint" ""
+		(property "Footprint" "Resistor_SMD:R_0805_2012Metric"
 			(at 164.338 33.02 90)
 			(effects
@@
 				)
 				(path "/83dee5c5-8c71-4ecf-8c4b-74a6ca3f5e87/7d7c01cb-e012-4aa5-8562-a4c629acedd9"
-					(reference "R22")
+					(reference "R47")
 					(unit 1)
 				)
@@
 			)
 		)
-		(property "Footprint" ""
+		(property "Footprint" "Capacitor_SMD:C_0805_2012Metric"
 			(at 73.9648 29.21 0)
 			(effects
@@
 			)
 		)
-		(property "Footprint" ""
+		(property "Footprint" "Resistor_SMD:R_0805_2012Metric"
 			(at 56.388 76.2 90)
 			(effects
@@
 			)
 		)
-		(property "Footprint" "PA107DP"
+		(property "Footprint" "pa107:PA107DP"
 			(at 90.17 158.42 0)
 			(effects
@@
 			)
 		)
-		(property "Footprint" ""
+		(property "Footprint" "Capacitor_SMD:C_0805_2012Metric"
 			(at 136.1948 48.26 0)
 			(effects
@@
 			)
 		)
-		(property "Footprint" ""
+		(property "Footprint" "Capacitor_THT:CP_Radial_D6.3mm_P2.50mm"
 			(at 148.8948 48.26 0)
 			(effects
@@
 			)
 		)
-		(property "Footprint" ""
+		(property "Footprint" "Capacitor_SMD:C_0805_2012Metric"
 			(at 90.4748 29.21 0)
 			(effects
@@
 			)
 		)
-		(property "Footprint" ""
+		(property "Footprint" "Capacitor_THT:CP_Radial_D6.3mm_P2.50mm"
 			(at 148.8948 29.21 0)
 			(effects
@@
 			)
 		)
-		(property "Footprint" ""
+		(property "Footprint" "Capacitor_SMD:C_0805_2012Metric"
 			(at 119.6848 29.21 0)
 			(effects
@@
 			)
 		)
-		(property "Footprint" ""
+		(property "Footprint" "Capacitor_SMD:C_0805_2012Metric"
 			(at 136.1948 29.21 0)
 			(effects

Commit message: sim the new lpf
Parts:
- added D4, D7: D, symbol Device:D
Connections:
- net GND: now also D4.2 (A), D7.1 (K)
- net PA_IN: now also D4.1 (K), D7.2 (A)

Commit message: routing draft 3
Parts:
- D4, D7: footprint (none) -> Diode_SMD:D_SOD-123
Changed lines of the file:
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@@
 			)
 		)
-		(property "Footprint" ""
+		(property "Footprint" "Diode_SMD:D_SOD-123"
 			(at 50.8 63.5 0)
 			(effects
@@
 			)
 		)
-		(property "Footprint" ""
+		(property "Footprint" "Diode_SMD:D_SOD-123"
 			(at 50.8 71.12 0)
 			(effects
